File: schematics_and_pcb/schematics_and_pcb.kicad_pcb (KiCad board)
At the start: 2 copper layers, 61.8 x 89.9 mm, 82 parts, among them J1 RND 205-00624, J2 RND 205-00627, J3 Motor con, J4 Conn_01x04_Male, J5 Conn_01x04_Male, J6 USB_OTG_custom, J7 i2c header, J8 i2c header, Q1 TSM2308CX RFG, SW1 RND 210-00210, SW2 SW_Push, U1 LP2985IM5-2.0/NOPB, U10 RND 135-00249, U11 RND 135-00249, U12 RND 135-00249, U2 TS3480CX33 RFG, U3 PWM3389DM-T3QU, U4 STM32F401RBTx, U5 LFXTAL055951, U6 9DB403DGLFT, U7 RND 135-00249, U8 RND 135-00249, U9 RND 135-00249

Commit message: fixed board
Parts:
- added G***: LOGO, LOGO, F.Cu at (119.0, 34.8)
- added G***: LOGO, LOGO, F.Cu at (69.5, 106.5)
- added G***: LOGO, LOGO, F.Cu at (71.0, 90.5)
- added G***: LOGO, LOGO, F.Cu at (96.0, 31.8)
- added G***: LOGO, LOGO, F.Cu at (126.2, 74.2)
- added G***: LOGO, LOGO, B.Cu at (126.5, 75.5)
- added G***: LOGO, LOGO, B.Cu at (128.2, 73.2)
- added J9: Conn_01x04_Male, Connector_PinHeader_1.00mm:PinHeader_1x04_P1.00mm_Vertical, F.Cu at (99.2, 70.0)
- R13, R16: value 680m -> 2.2
- R17: value 8.2 -> 22
- U6: value 9DB403DGLFT -> PCA9624
- moved C2 12.0 mm to (99.5, 82.2)
- moved R1 11.4 mm to (99.5, 78.5), turned to 90 degrees
- moved MOTION1 1.50 mm to (99.5, 86.5)
- moved R9 1.02 mm to (99.2, 73.0), turned to 90 degrees
- moved enc1 0.10 mm to (96.5, 44.3)
Connections:
- J5 pad 1: +5V -> VDDIO
Routing:
- net VDDIO: track 232.1 -> 276.9 mm, vias 16 -> 18
- net MOTION: track 30.2 -> 68.4 mm
- net +5V: track 243.0 -> 215.8 mm
- net VDD: track 64.5 -> 76.5 mm, vias 3 -> 2
- net SPI2_SCK: track 26.4 -> 38.1 mm, vias 0 -> 1
- net SPI2_MISO: track 31.6 -> 40.4 mm
- net SPI2_MOSI: track 30.5 -> 38.9 mm, vias 1 -> 0
- net SPI2_NCS: track 39.9 -> 35.4 mm, vias 2 -> 0
- net GND: track 115.5 -> 111.5 mm, vias 42 -> 39
- net PHASE_B: track 73.5 -> 71.0 mm
- net PHASE_A: track 72.5 -> 70.9 mm
- net LEFT_STATE: track 79.8 -> 79.0 mm
- net LEDP: track 3.09 -> 2.33 mm
- net BACK_STATE: track 45.7 -> 45.2 mm, vias 2 -> 1
Other:
- outline, holes or cut-outs redrawn
- board text added: "3v3"
- board text added: "Graphics by Elena Strineholm"
- board text added: "miso"
- board text added: "mosi"
- board text added: "ncs"
- board text added: "sck"
