File: schematics_and_pcb/Ivar_Erik_rev1.kicad_pcb (KiCad board)
At the start: 2 copper layers, 61.8 x 89.9 mm, 82 parts, among them J1 RND 205-00624, J2 RND 205-00627, J3 Motor con, J4 Conn_01x04_Male, J5 Conn_01x04_Male, J6 USB_OTG_custom, J7 i2c header, J8 i2c header, Q1 TSM2308CX RFG, SW1 RND 210-00210, SW2 SW_Push, U1 LP2985IM5-2.0/NOPB, U10 RND 135-00249, U11 RND 135-00249, U12 RND 135-00249, U2 TS3480CX33 RFG, U3 PWM3389DM-T3QU, U4 STM32F401RBTx, U5 LFXTAL055951, U6 9DB403DGLFT, U7 RND 135-00249, U8 RND 135-00249, U9 RND 135-00249

Commit message: fixed board
Parts:
- added G***: LOGO, LOGO, F.Cu at (119.0, 34.8)
- added G***: LOGO, LOGO, F.Cu at (69.5, 106.5)
- added G***: LOGO, LOGO, F.Cu at (71.0, 90.5)
- added G***: LOGO, LOGO, F.Cu at (96.0, 31.8)
- added G***: LOGO, LOGO, F.Cu at (126.2, 74.2)
- added G***: LOGO, LOGO, B.Cu at (126.5, 75.5)
- added G***: LOGO, LOGO, B.Cu at (128.2, 73.2)
- moved enc1 0.10 mm to (96.5, 44.3)
- renumbered 1v1 to 2v
Routing:
- net +5V: track 243.0 -> 232.1 mm
- net VDDR: track 34.2 -> 35.5 mm
Other:
- outline, holes or cut-outs redrawn
- board text added: "Graphics by Elena Strineholm"
