File: schematics_and_pcb/schematics_and_pcb.kicad_sch (KiCad schematic)
At the start: 82 parts, among them J1 RND 205-00624, J2 RND 205-00627, J3 Motor con, J4 Conn_01x04_Male, J5 Conn_01x04_Male, J6 USB_OTG_custom, J7 i2c header, J8 i2c header, Q1 TSM2308CX RFG, SW1 RND 210-00210, SW2 SW_Push, U1 LP2985IM5-2.0/NOPB, U10 RND 135-00249, U11 RND 135-00249, U12 RND 135-00249, U2 TS3480CX33 RFG, U3 PWM3389DM-T3QU, U4 STM32F401RBTx, U5 LFXTAL055951, U6 9DB403DGLFT, U7 RND 135-00249, U8 RND 135-00249, U9 RND 135-00249

Commit message: updated the bom
Parts:
- R13, R16: value 680m -> 2.2
- R17: value 8.2 -> 22
- U6: value 9DB403DGLFT -> PCA9624
Changed lines of the file:
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@@
     (in_bom yes) (on_board yes)
     (property "Reference" "R17" (id 0) (at 361.95 179.07 90))
-    (property "Value" "8.2" (id 1) (at 358.14 179.07 90))
+    (property "Value" "22" (id 1) (at 358.14 179.07 90))
     (property "Footprint" "Resistor_SMD:R_0805_2012Metric_Pad1.20x1.40mm_HandSolder" (id 2) (at 358.14 176.53 0)
       (effects (font (size 1.27 1.27)) hide)
@@
     (in_bom yes) (on_board yes) (fields_autoplaced)
     (property "Reference" "R13" (id 0) (at 358.14 165.1 90))
-    (property "Value" "680m" (id 1) (at 358.14 167.64 90))
+    (property "Value" "2.2" (id 1) (at 358.14 167.64 90))
     (property "Footprint" "Resistor_SMD:R_0805_2012Metric_Pad1.20x1.40mm_HandSolder" (id 2) (at 358.14 171.45 0)
       (effects (font (size 1.27 1.27)) hide)
@@
     (in_bom yes) (on_board yes) (fields_autoplaced)
     (property "Reference" "U6" (id 0) (at 302.895 156.21 0))
-    (property "Value" "9DB403DGLFT" (id 1) (at 302.895 158.75 0))
+    (property "Value" "PCA9624" (id 1) (at 302.895 158.75 0))
     (property "Footprint" "mouse:TSSOP-24" (id 2) (at 297.18 158.75 0)
       (effects (font (size 1.27 1.27)) hide)
@@
     (in_bom yes) (on_board yes)
     (property "Reference" "R16" (id 0) (at 354.33 173.99 90))
-    (property "Value" "680m" (id 1) (at 361.95 173.99 90))
+    (property "Value" "2.2" (id 1) (at 361.95 173.99 90))
     (property "Footprint" "Resistor_SMD:R_0805_2012Metric_Pad1.20x1.40mm_HandSolder" (id 2) (at 358.14 173.99 0)
       (effects (font (size 1.27 1.27)) hide)
@@
     )
     (path "/792a157e-cb19-4864-93f9-71633a825461"
-      (reference "R13") (unit 1) (value "680m") (footprint "Resistor_SMD:R_0805_2012Metric_Pad1.20x1.40mm_HandSolder")
+      (reference "R13") (unit 1) (value "2.2") (footprint "Resistor_SMD:R_0805_2012Metric_Pad1.20x1.40mm_HandSolder")
     )
     (path "/2a4d6102-d0e4-47d6-81b6-8da78f401505"
@@
     )
     (path "/ce63bba4-4792-49bb-991f-eed6095c7f6a"
-      (reference "R16") (unit 1) (value "680m") (footprint "Resistor_SMD:R_0805_2012Metric_Pad1.20x1.40mm_HandSolder")
+      (reference "R16") (unit 1) (value "2.2") (footprint "Resistor_SMD:R_0805_2012Metric_Pad1.20x1.40mm_HandSolder")
     )
     (path "/14d53526-2ffb-4d05-8740-bfc9da25797b"
-      (reference "R17") (unit 1) (value "8.2") (footprint "Resistor_SMD:R_0805_2012Metric_Pad1.20x1.40mm_HandSolder")
+      (reference "R17") (unit 1) (value "22") (footprint "Resistor_SMD:R_0805_2012Metric_Pad1.20x1.40mm_HandSolder")
     )
     (path "/d66de268-e697-4036-b690-c8e2d2ae5ff7"
@@
     )
     (path "/a2ee253e-ed9e-42e6-96e3-d788a584d3c0"
-      (reference "U6") (unit 1) (value "9DB403DGLFT") (footprint "mouse:TSSOP-24")
+      (reference "U6") (unit 1) (value "PCA9624") (footprint "mouse:TSSOP-24")
     )
     (path "/0e677c85-3782-4cac-898b-a79bb3ec6e2d"

Commit message: fixed board
Parts:
- added J9: Conn_01x04_Male, Connector_PinHeader_1.00mm:PinHeader_1x04_P1.00mm_Vertical, symbol Connector:Conn_01x04_Male
Connections:
- net +3V3: now also J5.1 (Pin_1)
- net +5V: no longer J5.1 (Pin_1)
- net SPI2_MISO: now also J9.2 (Pin_2)
- net SPI2_MOSI: now also J9.3 (Pin_3)
- net SPI2_NCS: now also J9.1 (Pin_1)
- net SPI2_SCK: now also J9.4 (Pin_4)
Other:
- note added: "C18 is wrong"
Changed lines of the file:
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@@
     (effects (font (size 5 5)) (justify left bottom))
   )
+  (text "C18 is wrong\n\n" (at 165.1 72.39 0)
+    (effects (font (size 1.27 1.27)) (justify left bottom))
+  )
   (text "FRONT BUTTONS\n" (at 12.7 207.01 0)
     (effects (font (size 5 5)) (justify left bottom))
@@
     )
   )
+  (global_label "SPI2_MOSI" (shape output) (at 109.22 143.51 180) (fields_autoplaced)
+    (effects (font (size 1.27 1.27)) (justify right))
+    (property "Intersheet References" "${INTERSHEET_REFS}" (id 0) (at 96.9493 143.4306 0)
+      (effects (font (size 1.27 1.27)) (justify right) hide)
+    )
+  )
   (global_label "PHASE_A" (shape output) (at 356.87 66.04 0) (fields_autoplaced)
     (effects (font (size 1 1)) (justify left))
@@
     )
   )
+  (global_label "SPI2_SCK" (shape output) (at 109.22 140.97 180) (fields_autoplaced)
+    (effects (font (size 1.27 1.27)) (justify right))
+    (property "Intersheet References" "${INTERSHEET_REFS}" (id 0) (at 97.7959 141.0494 0)
+      (effects (font (size 1.27 1.27)) (justify right) hide)
+    )
+  )
   (global_label "PWM6" (shape output) (at 311.15 182.88 0) (fields_autoplaced)
     (effects (font (size 1.27 1.27)) (justify left))
@@
     )
   )
+  (global_label "SPI2_MISO" (shape input) (at 109.22 146.05 180) (fields_autoplaced)
+    (effects (font (size 1.27 1.27)) (justify right))
+    (property "Intersheet References" "${INTERSHEET_REFS}" (id 0) (at 96.9493 145.9706 0)
+      (effects (font (size 1.27 1.27)) (justify right) hide)
+    )
+  )
   (global_label "VDDB" (shape output) (at 364.49 171.45 0) (fields_autoplaced)
     (effects (font (size 1.27 1.27)) (justify left))
@@
     )
   )
+  (global_label "SPI2_NCS" (shape output) (at 109.22 148.59 180) (fields_autoplaced)
+    (effects (font (size 1.27 1.27)) (justify right))
+    (property "Intersheet References" "${INTERSHEET_REFS}" (id 0) (at 97.7355 148.6694 0)
+      (effects (font (size 1.27 1.27)) (justify right) hide)
+    )
+  )
   (global_label "BOOT0" (shape input) (at 36.83 149.86 0) (fields_autoplaced)
     (effects (font (size 1.27 1.27)) (justify left))
@@
   )
   (symbol (lib_id "Device:C_Small") (at 195.58 69.85 270) (unit 1)
-    (in_bom yes) (on_board yes) (fields_autoplaced)
+    (in_bom yes) (on_board yes)
     (property "Reference" "C18" (id 0) (at 196.8438 72.39 0)
       (effects (font (size 1.27 1.27)) (justify left))
@@
     (pin "2")
   )
+  (symbol (lib_id "power:+3V3") (at 156.21 134.62 180) (unit 1)
+    (in_bom yes) (on_board yes) (fields_autoplaced)
+    (property "Reference" "#PWR?" (id 0) (at 156.21 130.81 0)
+      (effects (font (size 1.27 1.27)) hide)
+    )
+    (property "Value" "+3V3" (id 1) (at 156.21 139.7 0))
+    (property "Footprint" "" (id 2) (at 156.21 134.62 0)
+      (effects (font (size 1.27 1.27)) hide)
+    )
+    (property "Datasheet" "" (id 3) (at 156.21 134.62 0)
+      (effects (font (size 1.27 1.27)) hide)
+    )
+    (pin "1")
+  )
   (symbol (lib_id "power:GND") (at 325.12 175.26 0) (unit 1)
     (in_bom yes) (on_board yes) (fields_autoplaced)
@@
     (pin "2")
   )
-  (symbol (lib_id "power:+5V") (at 156.21 134.62 180) (unit 1)
-    (in_bom yes) (on_board yes)
-    (property "Reference" "#PWR0162" (id 0) (at 156.21 130.81 0)
-      (effects (font (size 1.27 1.27)) hide)
-    )
-    (property "Value" "+5V" (id 1) (at 156.21 139.7 90))
-    (property "Footprint" "" (id 2) (at 156.21 134.62 0)
-      (effects (font (size 1.27 1.27)) hide)
-    )
-    (property "Datasheet" "" (id 3) (at 156.21 134.62 0)
-      (effects (font (size 1.27 1.27)) hide)
-    )
-    (pin "1")
-  )
   (symbol (lib_id "power:+3V3") (at 113.03 27.94 0) (unit 1)
     (in_bom yes) (on_board yes) (fields_autoplaced)
@@
     (pin "2")
   )
+  (symbol (lib_id "Connector:Conn_01x04_Male") (at 114.3 146.05 180) (unit 1)
+    (in_bom yes) (on_board yes) (fields_autoplaced)
+    (property "Reference" "J9" (id 0) (at 115.57 143.5099 0)
+      (effects (font (size 1.27 1.27)) (justify right))
+    )
+    (property "Value" "Conn_01x04_Male" (id 1) (at 115.57 146.0499 0)
+      (effects (font (size 1.27 1.27)) (justify right))
+    )
+    (property "Footprint" "Connector_PinHeader_1.00mm:PinHeader_1x04_P1.00mm_Vertical" (id 2) (at 114.3 146.05 0)
+      (effects (font (size 1.27 1.27)) hide)
+    )
+    (property "Datasheet" "~" (id 3) (at 114.3 146.05 0)
+      (effects (font (size 1.27 1.27)) hide)
+    )
+    (pin "1")
+    (pin "2")
+    (pin "3")
+    (pin "4")
+  )
   (symbol (lib_id "Device:R_Small") (at 96.52 189.23 180) (unit 1)
     (in_bom yes) (on_board yes)
@@
       (reference "#PWR0161") (unit 1) (value "GND") (footprint "")
     )
-    (path "/ad7960f0-0ffb-4b70-abfd-f55fb0c91327"
-      (reference "#PWR0162") (unit 1) (value "+5V") (footprint "")
-    )
     (path "/0d64b0b3-99f7-47aa-8827-29913ce2edcb"
       (reference "#PWR0163") (unit 1) (value "GND") (footprint "")
@@
       (reference "#PWR0184") (unit 1) (value "+3V3") (footprint "")
     )
+    (path "/73c1b947-11e9-40cf-af03-56c22766304e"
+      (reference "#PWR?") (unit 1) (value "+3V3") (footprint "")
+    )
     (path "/22579084-dfa4-4d73-996e-5c94c7085cc5"
       (reference "1v1") (unit 1) (value "1v94_TEST") (footprint "Connector_PinHeader_2.54mm:PinHeader_1x01_P2.54mm_Vertical")
@@
       (reference "J8") (unit 1) (value "i2c header") (footprint "Connector_PinHeader_2.54mm:PinHeader_1x04_P2.54mm_Vertical")
     )
+    (path "/c0f49285-51e4-4689-9a15-7f7a4f2ae40a"
+      (reference "J9") (unit 1) (value "Conn_01x04_Male") (footprint "Connector_PinHeader_1.00mm:PinHeader_1x04_P1.00mm_Vertical")
+    )
     (path "/fd975609-7adf-48bb-bc3e-84d8eed1717e"
